Commit message: big/bang-initial version

File: kvn_robot_description/urdf/kvn_rover.urdf.xacro (robot description, xacro)
@@ -10,4 +10,5 @@
   <xacro:include
     filename="$(find kvn_robot_description)/urdf/kvn_rover/kvn_rover_macro.ros2_control.xacro" />
+  <xacro:include filename="$(find kvn_robot_description)/urdf/gazebo/gazebo.xacro" />
   <xacro:property name="props_yaml" value="$(find kvn_robot_description)/config/robot_config.yaml" />
   <xacro:property name="robot_props" value="${xacro.load_yaml(props_yaml)}" />

File: kvn_robot_description/urdf/kvn_rover/kvn_rover_macro.ros2_control.xacro (robot description, xacro)
@@ -2,5 +2,5 @@
 <robot xmlns:xacro="http://wiki.ros.org/xacro">
   <xacro:macro name="ds210_joint" params="name id">
-      <joint name="£{name}">
+      <joint name="${name}">
         <command_interface name="velocity"/>
         <command_interface name="effort"/>
@@ -32,8 +32,8 @@
         </xacro:unless>
       </hardware>
-      <xacro:ds210_joint name="${prefix}joint1" id="16"/>
-      <xacro:ds210_joint name="${prefix}joint2" id="17"/>
-      <xacro:ds210_joint name="${prefix}joint3" id="18"/>
-      <xacro:ds210_joint name="${prefix}joint4" id="19"/>
+      <xacro:ds210_joint name="${prefix}front_left_joint" id="16"/>
+      <xacro:ds210_joint name="${prefix}front_right_joint" id="17"/>
+      <xacro:ds210_joint name="${prefix}back_left_joint" id="18"/>
+      <xacro:ds210_joint name="${prefix}back_right_joint" id="19"/>
     </ros2_control>
     <xacro:if value="$(arg sim_gazebo)">
